Commit message: Fixed map issue and camera orientation

File: catkin_ws/src/my_robot/urdf/project_robot.xacro (robot description, xacro)
@@ -155,5 +155,5 @@
   </link>
   <joint name="camera_optical_joint" type="fixed">
-    <origin xyz="0 0 0" rpy="-1.5707 0 -1.5707"/>
+    <origin xyz="0 0 0" rpy="0 0 0"/>
     <parent link="camera"/>
     <child link="camera_link_optical"/>
